File: Electrical/Test Boards/WT32i_Breakout/WT32i_Breakout.sch (KiCad schematic (older format))
At the start: 14 parts, among them P1 Stereo_Audio_Jack_3.5mm, P2 CONN_02X03, P3 CONN_01X06, P4 CONN_01X06, P5 CONN_01X02, U2 TPS79933

Commit message: Test board updates
Parts:
- removed P1: Stereo_Audio_Jack_3.5mm, lib:CUI_Stereo_Audio_Jack, symbol Stereo_Audio_Jack_3.5mm
- removed P2: CONN_02X03, Socket_Strips:Socket_Strip_Straight_2x03, symbol CONN_02X03
- removed P3, P4: CONN_01X06, Socket_Strips:Socket_Strip_Straight_1x06, symbol CONN_01X06
- removed P5: CONN_01X02, Socket_Strips:Socket_Strip_Straight_1x02, symbol CONN_01X02
- removed U?: WT32i-RESCUE-WT32i_Breakout, symbol WT32i-RESCUE-WT32i_Breakout
- added D2: CONN_LED, symbol Led_Small
- added D3: PWR_LED, symbol Led_Small
- added P1: UART_CONN, symbol CONN_01X06
- added P3: POWER_CONN, symbol CONN_01X02
- added P4: Stereo_Audio_Jack_3.5mm, symbol Stereo_Audio_Jack_3.5mm
- added P?: CONN_01X04, symbol CONN_01X04
- added R3, R4: R_Small, symbol R_Small
- added U1: WT32i, symbol WT32i
- C1, C2: footprint Capacitors_SMD:C_0603 -> (none)
- C3, C4: value 330uF -> CP1_Small; footprint Capacitors_Tantalum_SMD:TantalC_SizeD_EIA-7343_Reflow -> (none)
- D1: footprint Diodes_SMD:SOD-123 -> (none)
- R1, R2: value 1M -> R_Small; footprint Resistors_SMD:R_0603 -> (none)
- U2: footprint TO_SOT_Packages_SMD:SOT-23-5 -> (none)
Connections:
- net labels added: +3V3, I2S_IN, I2S_OUT, I2S_SCK, I2S_WS, RESET
- net labels removed: +3.3V, FTDI_CTS, FTDI_RTS, ON/OFF_FROM_HOST, RESET_FROM_HOST, SPI_CLK, SPI_CS, SPI_MISO, SPI_MOSI, UART_NCTS, UART_NRTS
- wire segments 64 -> 39
- no-connect marks 3 -> 4

Commit message: Test board updates
Parts:
- gave numbers to parts that had none: 1
Connections:
- wire segments 39 -> 43
Changed lines of the file:
@@
 Sheet 1 1
 Title "WT32i Breakout"
-Date "2016-06-02"
+Date "2016-06-10"
 Rev "2.0"
 Comp "Noctivore"
@@
 	3050 3300 3050 3250
 $Comp
-L CONN_01X04 P?
+L CONN_01X04 P2
 U 1 1 5750CB3B
-P 7600 3950
-F 0 "P?" H 7600 4200 50  0000 C CNN
-F 1 "CONN_01X04" V 7700 3950 50  0000 C CNN
-F 2 "" H 7600 3950 50  0000 C CNN
-F 3 "" H 7600 3950 50  0000 C CNN
-	1    7600 3950
-	1    0    0    -1
-$EndComp
+P 7850 3950
+F 0 "P2" H 7850 4200 50  0000 C CNN
+F 1 "CONN_01X04" V 7950 3950 50  0000 C CNN
+F 2 "" H 7850 3950 50  0000 C CNN
+F 3 "" H 7850 3950 50  0000 C CNN
+	1    7850 3950
+	1    0    0    -1
+$EndComp
+Wire Wire Line
+	7550 3800 7650 3800
+Wire Wire Line
+	7550 3900 7650 3900
+Wire Wire Line
+	7550 4000 7650 4000
+Wire Wire Line
+	7550 4100 7650 4100
+Text Label 7550 3800 2    60   ~ 0
+I2S_IN
+Text Label 7550 3900 2    60   ~ 0
+I2S_OUT
+Text Label 7550 4000 2    60   ~ 0
+I2S_WS
+Text Label 7550 4100 2    60   ~ 0
+I2S_SCK
 $EndSCHEMATC
