File: Electrical/Test Boards/WT32i_Breakout/WT32i_Breakout.sch (KiCad schematic (older format))
At the start: 17 parts, among them P1 UART_CONN, P2 CONN_01X04, P3 POWER_CONN, P4 Stereo_Audio_Jack_3.5mm, U1 WT32i, U2 TPS79933

Commit message: WT32i test board updates
Parts:
- removed P3: POWER_CONN, symbol CONN_01X02
- added C5, C6: 33pF, Capacitors_SMD:C_0603, symbol C_Small
- added L1, L2: 33uH, Capacitors_SMD:C_0402, symbol L_Small
- added P3: PWR_CONN, Socket_Strips:Socket_Strip_Straight_1x03, symbol CONN_01X03
- C1, C2: footprint (none) -> Capacitors_SMD:C_0603
- C3, C4: value CP1_Small -> 330uF/6.3V; footprint (none) -> Capacitors_Tantalum_SMD:TantalC_SizeD_EIA-7343_Reflow
- D1: value D_Small -> D_Reset; footprint (none) -> Diodes_SMD:SOD-123
- D2, D3: footprint (none) -> LEDs:LED_0603
- P1: footprint (none) -> Socket_Strips:Socket_Strip_Straight_1x06
- P2: value CONN_01X04 -> I2S_CONN; footprint (none) -> Socket_Strips:Socket_Strip_Straight_1x04
- P4: footprint (none) -> wt32i_breakout:CUI_Stereo_Audio_Jack
- R1: value R_Small -> 100; footprint (none) -> Resistors_SMD:R_0603
- R2: value R_Small -> 820; footprint (none) -> Resistors_SMD:R_0603
- R3, R4: value R_Small -> 1M; footprint (none) -> Resistors_SMD:R_0603
- U1: footprint (none) -> wt32i_breakout:WT32i
- U2: footprint (none) -> TO_SOT_Packages_SMD:SOT-23-5
Connections:
- wire segments 43 -> 71

Commit message: WT32i test board updates
Parts:
- added P5: AGND, Socket_Strips:Socket_Strip_Straight_1x01, symbol CONN_01X01
Connections:
- net labels added: GNDA
- wire segments 71 -> 72
Other:
- note added: "AGND goes to Pin1\nof UART_CONN P1\nfor clean return path\nto GND for Audio Jack"

Commit message: WT32i test board updates
Parts:
- removed D1: D_Reset, Diodes_SMD:SOD-123, symbol D_Small
- removed P3: PWR_CONN, Socket_Strips:Socket_Strip_Straight_1x03, symbol CONN_01X03
- removed P5: AGND, Socket_Strips:Socket_Strip_Straight_1x01, symbol CONN_01X01
- added P3: PWR_CONN, Socket_Strips:Socket_Strip_Straight_1x02, symbol CONN_01X02
Connections:
- net labels removed: RESET
- wire segments 72 -> 68
- no-connect marks 4 -> 5
Other:
- note removed: "AGND goes to Pin1\nof UART_CONN P1\nfor clean return path\nto GND for Audio Jack"
Changed lines of the file:
@@
 Sheet 1 1
 Title "WT32i Breakout"
-Date "2016-06-17"
+Date "2016-06-19"
 Rev "2.0"
 Comp "Noctivore"
@@
 $EndComp
 $Comp
-L D_Small D1
-U 1 1 57509CCB
-P 4100 4250
-F 0 "D1" H 4050 4330 50  0000 L CNN
-F 1 "D_Reset" H 3950 4170 50  0000 L CNN
-F 2 "Diodes_SMD:SOD-123" V 4100 4250 50  0001 C CNN
-F 3 "" V 4100 4250 50  0000 C CNN
-	1    4100 4250
-	-1   0    0    1
-$EndComp
-$Comp
 L Led_Small D2
 U 1 1 57509D21
@@
 	1    0    0    -1
 $EndComp
-Text Label 3900 4250 2    60   ~ 0
-RESET
 Text Label 5950 3350 0    60   ~ 0
 I2S_IN
@@
 L GND #PWR016
 U 1 1 5750C81D
-P 3100 4050
-F 0 "#PWR016" H 3100 3800 50  0001 C CNN
-F 1 "GND" H 3100 3900 50  0000 C CNN
-F 2 "" H 3100 4050 50  0000 C CNN
-F 3 "" H 3100 4050 50  0000 C CNN
-	1    3100 4050
+P 3100 4000
+F 0 "#PWR016" H 3100 3750 50  0001 C CNN
+F 1 "GND" H 3100 3850 50  0000 C CNN
+F 2 "" H 3100 4000 50  0000 C CNN
+F 3 "" H 3100 4000 50  0000 C CNN
+	1    3100 4000
 	1    0    0    -1
 $EndComp
@@
 L +3V3 #PWR017
 U 1 1 5750C858
-P 3100 3750
-F 0 "#PWR017" H 3100 3600 50  0001 C CNN
-F 1 "+3V3" H 3100 3890 50  0000 C CNN
-F 2 "" H 3100 3750 50  0000 C CNN
-F 3 "" H 3100 3750 50  0000 C CNN
-	1    3100 3750
+P 3100 3800
+F 0 "#PWR017" H 3100 3650 50  0001 C CNN
+F 1 "+3V3" H 3100 3940 50  0000 C CNN
+F 2 "" H 3100 3800 50  0000 C CNN
+F 3 "" H 3100 3800 50  0000 C CNN
+	1    3100 3800
 	1    0    0    -1
 $EndComp
@@
 Text Label 7550 4650 2    60   ~ 0
 I2S_SCK
-$Comp
-L CONN_01X03 P3
-U 1 1 575DE97A
-P 2850 3900
-F 0 "P3" H 2850 4100 50  0000 C CNN
-F 1 "PWR_CONN" V 2950 3900 50  0000 C CNN
-F 2 "Socket_Strips:Socket_Strip_Straight_1x03" H 2850 3900 50  0001 C CNN
-F 3 "" H 2850 3900 50  0000 C CNN
-	1    2850 3900
-	-1   0    0    1
-$EndComp
-Text Label 3150 3900 0    60   ~ 0
-RESET
 $Comp
 L GND #PWR018
@@
 	3700 4750 3700 4550
 Wire Wire Line
-	4200 4250 4400 4250
-Wire Wire Line
-	3900 4250 4000 4250
-Wire Wire Line
 	2800 2750 2800 3050
 Wire Wire Line
 	2800 3250 2800 3300
 Wire Wire Line
-	3050 4000 3100 4000
-Wire Wire Line
-	3100 4000 3100 4050
-Wire Wire Line
-	3050 3800 3100 3800
-Wire Wire Line
-	3100 3800 3100 3750
+	3050 3850 3100 3850
+Wire Wire Line
+	3100 3850 3100 3800
 Wire Wire Line
 	7550 4350 7650 4350
@@
 Wire Wire Line
 	7550 4650 7650 4650
-Wire Wire Line
-	3150 3900 3050 3900
 Wire Wire Line
 	4400 4050 4050 4050
@@
 	7500 2850 7500 2950
 Connection ~ 7500 2950
-$Comp
-L GNDA #PWR021
-U 1 1 5764D154
-P 8900 3900
-F 0 "#PWR021" H 8900 3650 50  0001 C CNN
-F 1 "GNDA" H 8900 3750 50  0000 C CNN
-F 2 "" H 8900 3900 50  0000 C CNN
-F 3 "" H 8900 3900 50  0000 C CNN
-	1    8900 3900
-	1    0    0    -1
-$EndComp
-$Comp
-L CONN_01X01 P5
-U 1 1 5764D9DF
-P 8900 3600
-F 0 "P5" H 8900 3700 50  0000 C CNN
-F 1 "AGND" V 9000 3600 50  0000 C CNN
-F 2 "Socket_Strips:Socket_Strip_Straight_1x01" H 8900 3600 50  0001 C CNN
-F 3 "" H 8900 3600 50  0000 C CNN
-	1    8900 3600
-	0    -1   -1   0
-$EndComp
-Wire Wire Line
-	8900 3800 8900 3900
-Text Notes 7700 4050 0    60   ~ 0
-AGND goes to Pin1\nof UART_CONN P1\nfor clean return path\nto GND for Audio Jack
+NoConn ~ 4400 4250
+$Comp
+L CONN_01X02 P3
+U 1 1 576782E6
+P 2850 3900
+F 0 "P3" H 2850 4050 50  0000 C CNN
+F 1 "PWR_CONN" V 2950 3900 50  0000 C CNN
+F 2 "Socket_Strips:Socket_Strip_Straight_1x02" H 2850 3900 50  0001 C CNN
+F 3 "" H 2850 3900 50  0000 C CNN
+	1    2850 3900
+	-1   0    0    1
+$EndComp
+Wire Wire Line
+	3050 3950 3100 3950
+Wire Wire Line
+	3100 3950 3100 4000
 $EndSCHEMATC

Commit message: WT32i test board updates
Parts:
- L1, L2: value 33uH -> 33nH
Changed lines of the file:
@@
 Sheet 1 1
 Title "WT32i Breakout"
-Date "2016-06-19"
+Date "2016-07-10"
 Rev "2.0"
 Comp "Noctivore"
@@
 P 7200 2950
 F 0 "L1" H 7230 2990 50  0000 L CNN
-F 1 "33uH" H 7230 2910 50  0000 L CNN
+F 1 "33nH" H 7230 2910 50  0000 L CNN
 F 2 "Capacitors_SMD:C_0402" H 7200 2950 50  0001 C CNN
 F 3 "" H 7200 2950 50  0000 C CNN
@@
 P 7200 3150
 F 0 "L2" H 7230 3190 50  0000 L CNN
-F 1 "33uH" H 7230 3110 50  0000 L CNN
+F 1 "33nH" H 7230 3110 50  0000 L CNN
 F 2 "Capacitors_SMD:C_0402" H 7200 3150 50  0001 C CNN
 F 3 "" H 7200 3150 50  0000 C CNN
