File: Electrical/Test Boards/WT32i_Breakout/WT32i_Breakout.kicad_pcb (KiCad board)
At the start: 2 copper layers, 56.4 x 30.5 mm, 22 parts, among them P1 UART_CONN, P2 I2S_CONN, P3 PWR_CONN, P4 Stereo_Audio_Jack_3.5mm, P5 AGND, U1 WT32i, U2 TPS79933

Commit message: WT32i test board updates
Parts:
- removed D1: D_Reset, Diodes_SMD:SOD-123
- removed P5: AGND, wt32i_breakout:AGND
- added REF**: VIA, wt32i_breakout:VIA, F.Cu at (148.7, 79.1)
- added REF**: VIA, wt32i_breakout:VIA, F.Cu at (131.3, 100.4)
- added REF**: VIA, wt32i_breakout:VIA, F.Cu at (122.0, 104.0)
- added REF**: VIA, wt32i_breakout:VIA, F.Cu at (119.0, 104.0)
- added REF**: VIA, wt32i_breakout:VIA, F.Cu at (114.7, 103.0)
- added REF**: VIA, wt32i_breakout:VIA, F.Cu at (111.7, 104.5)
- added REF**: VIA, wt32i_breakout:VIA, F.Cu at (111.3, 101.3)
- added REF**: VIA, wt32i_breakout:VIA, F.Cu at (108.1, 103.0)
- added REF**: VIA, wt32i_breakout:VIA, F.Cu at (112.2, 88.8)
- added REF**: VIA, wt32i_breakout:VIA, F.Cu at (119.1, 86.4)
- added REF**: VIA, wt32i_breakout:VIA, F.Cu at (115.5, 86.4)
- added REF**: VIA, wt32i_breakout:VIA, F.Cu at (144.5, 79.1)
- added REF**: VIA, wt32i_breakout:VIA, F.Cu at (115.5, 85.4)
- added REF**: VIA, wt32i_breakout:VIA, F.Cu at (148.7, 88.6)
- added REF**: VIA, wt32i_breakout:VIA, F.Cu at (144.5, 88.6)
- added REF**: VIA, wt32i_breakout:VIA, F.Cu at (131.2, 83.4)
- added REF**: VIA, wt32i_breakout:VIA, F.Cu at (134.8, 83.4)
- added REF**: VIA, wt32i_breakout:VIA, F.Cu at (134.8, 88.4)
- added REF**: VIA, wt32i_breakout:VIA, F.Cu at (131.2, 88.4)
- added REF**: VIA, wt32i_breakout:VIA, F.Cu at (131.2, 92.4)
- P3: footprint Socket_Strips:Socket_Strip_Straight_1x03 -> Socket_Strips:Socket_Strip_Straight_1x02
- moved P3 2.56 mm to (112.0, 80.0)
- moved R2 1.25 mm to (113.5, 104.5)
- moved D3 1.06 mm to (116.4, 104.5)
- moved R1 0.42 mm to (113.5, 89.5)
- moved D2 0.38 mm to (113.5, 92.6)
- moved P1 0.27 mm to (109.0, 84.5)
Connections:
- P3 pad 2: /RESET -> +3V3
Routing:
- net GNDA: track 0.00 -> 55.7 mm, vias 0 -> 1
- net +3V3: track 23.0 -> 53.0 mm
- net +5V: track 5.71 -> 17.9 mm, vias 0 -> 1
- net /UART_RXD: track 0.00 -> 10.9 mm
- net /UART_TXD: track 0.00 -> 10.3 mm
- net GND: track 0.00 -> 5.69 mm
- net Net-(D2-Pad2): track 0.00 -> 3.80 mm
- net Net-(D2-Pad1): track 0.00 -> 1.62 mm
- net Net-(D3-Pad1): track 0.00 -> 1.43 mm
Other:
- board text added: "3V3"
- board text added: "5V"
- board text added: "CONN"
- board text added: "GND"
- board text added: "I2S:"
- board text added: "IN"
- board text added: "LEFT"
- board text added: "OUT"
- board text added: "PWR"
- board text added: "RIGHT"
- board text added: "RX"
- board text added: "SCK"
- board text added: "TX"
- board text added: "WS"

Commit message: gerber/README updates
Routing:
- net GNDA: track 55.7 -> 19.0 mm
- net GND: track 5.69 -> 42.4 mm
Changed lines of the file:
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@@
   (page A4)
   (title_block
-    (date 2016-06-17)
+    (date 2016-06-22)
   )
   (layers
@@
     (visible_elements FFFFFF7F)
     (pcbplotparams
-      (layerselection 0x000f8_80000001)
+      (layerselection 0x010f8_80000001)
       (usegerberextensions true)
       (excludeedgelayer true)
@@
   (segment (start 109.1524 84.5) (end 109 84.5) (width 0.5) (layer B.Cu) (net 2))
   (segment (start 112.25 87.5976) (end 112.25 88.75) (width 0.5) (layer B.Cu) (net 2))
+  (segment (start 141.51 80.16) (end 134.3 87.37) (width 0.5) (layer B.Cu) (net 2))
+  (segment (start 111.7 84.5) (end 109 84.5) (width 0.5) (layer B.Cu) (net 2))
+  (segment (start 134.3 87.37) (end 114.57 87.37) (width 0.5) (layer B.Cu) (net 2))
+  (segment (start 114.57 87.37) (end 111.7 84.5) (width 0.5) (layer B.Cu) (net 2))
   (segment (start 117.175 100.37) (end 117.175 104.4957) (width 0.4) (layer F.Cu) (net 3))
   (segment (start 117.175 104.4957) (end 117.1793 104.5) (width 0.25) (layer F.Cu) (net 3))
@@
   (segment (start 131.55 102.325) (end 132.62 103.395) (width 0.4) (layer F.Cu) (net 20))
   (segment (start 155.9 80.16) (end 141.51 80.16) (width 0.5) (layer B.Cu) (net 25))
-  (segment (start 141.51 80.16) (end 134.3 87.37) (width 0.5) (layer B.Cu) (net 25))
-  (segment (start 111.7 84.5) (end 109 84.5) (width 0.5) (layer B.Cu) (net 25))
-  (segment (start 134.3 87.37) (end 114.57 87.37) (width 0.5) (layer B.Cu) (net 25))
-  (segment (start 114.57 87.37) (end 111.7 84.5) (width 0.5) (layer B.Cu) (net 25))
   (segment (start 155.9 80.16) (end 160.49 80.16) (width 0.5) (layer F.Cu) (net 25))
   (segment (start 160.49 80.16) (end 160.5 80.17) (width 0.25) (layer F.Cu) (net 25))

Commit message: WT32i test board updates
Parts:
- L1, L2: value 33uH -> 33nH
Routing:
- net GNDA: track 19.0 -> 4.60 mm, vias 1 -> 0
- net GND: track 42.4 -> 56.8 mm, vias 0 -> 1
Changed lines of the file:
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@@
   (page A4)
   (title_block
-    (date 2016-06-22)
+    (date 2016-07-10)
   )
   (layers
@@
       (effects (font (size 1 1) (thickness 0.15)))
     )
-    (fp_text value 33uH (at 0 1.7) (layer F.Fab) hide
+    (fp_text value 33nH (at 0 1.7) (layer F.Fab) hide
       (effects (font (size 1 1) (thickness 0.15)))
     )
@@
       (effects (font (size 1 1) (thickness 0.15)))
     )
-    (fp_text value 33uH (at 0 1.7 180) (layer F.Fab) hide
+    (fp_text value 33nH (at 0 1.7 180) (layer F.Fab) hide
       (effects (font (size 1 1) (thickness 0.15)))
     )
@@
   (segment (start 134.3 87.37) (end 114.57 87.37) (width 0.5) (layer B.Cu) (net 2))
   (segment (start 114.57 87.37) (end 111.7 84.5) (width 0.5) (layer B.Cu) (net 2))
+  (segment (start 155.9 80.16) (end 141.51 80.16) (width 0.5) (layer B.Cu) (net 2))
+  (via (at 155.9 80.16) (size 0.6) (drill 0.4) (layers F.Cu B.Cu) (net 2))
   (segment (start 117.175 100.37) (end 117.175 104.4957) (width 0.4) (layer F.Cu) (net 3))
   (segment (start 117.175 104.4957) (end 117.1793 104.5) (width 0.25) (layer F.Cu) (net 3))
@@
   (segment (start 131 102.325) (end 131.55 102.325) (width 0.4) (layer F.Cu) (net 20))
   (segment (start 131.55 102.325) (end 132.62 103.395) (width 0.4) (layer F.Cu) (net 20))
-  (segment (start 155.9 80.16) (end 141.51 80.16) (width 0.5) (layer B.Cu) (net 25))
   (segment (start 155.9 80.16) (end 160.49 80.16) (width 0.5) (layer F.Cu) (net 25))
   (segment (start 160.49 80.16) (end 160.5 80.17) (width 0.25) (layer F.Cu) (net 25))
-  (via (at 155.9 80.16) (size 0.6) (drill 0.4) (layers F.Cu B.Cu) (net 25))
   (zone (net 2) (net_name GND) (layer F.Cu) (hatch edge 0.508)
     (connect_pads (clearance 0.381))
