File: Electrical/Test Boards/Lights_Breakout/Lights_Breakout.kicad_pcb (KiCad board)
At the start: 2 copper layers, 22 x 18 mm, 5 parts, among them P1 LIGHTS_HEADER, P2 SIGNAL_HEADER, Q1 IPD30N06S2L23ATMA3

Commit message: Lights test board corrections
Parts:
- Q1: value IPD30N06S2L23ATMA3 -> IPD30N06S2L-23
Connections:
- P1 pad 1: +12V -> GND
Other:
- board text added: "GND"
- board text added: "LIGHTS"
- board text added: "SIG"
Changed lines of the file:
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@@
 (kicad_pcb (version 4) (host pcbnew 4.0.2+e4-6225~38~ubuntu15.04.1-stable)
   (general
-    (links 7)
-    (no_connects 0)
+    (links 8)
+    (no_connects 1)
     (area 132.924999 90.924999 155.075001 109.075001)
     (thickness 1.6)
-    (drawings 10)
+    (drawings 14)
     (tracks 9)
     (zones 0)
     (modules 5)
-    (nets 6)
+    (nets 5)
   )
   (page A4)
   (title_block
-    (date 2016-06-22)
+    (date 2016-07-09)
   )
   (layers
@@
   )
   (net 0 "")
-  (net 1 +12V)
-  (net 2 "Net-(P1-Pad2)")
-  (net 3 GND)
-  (net 4 "Net-(P2-Pad2)")
-  (net 5 "Net-(Q1-Pad1)")
+  (net 1 "Net-(P1-Pad2)")
+  (net 2 GND)
+  (net 3 "Net-(P2-Pad2)")
+  (net 4 "Net-(Q1-Pad1)")
   (net_class Default "This is the default net class."
     (clearance 0.2)
@@
     (uvia_dia 0.3)
     (uvia_drill 0.1)
-    (add_net +12V)
     (add_net GND)
     (add_net "Net-(P1-Pad2)")
@@
     (fp_line (start 7.5 3.7) (end -7.5 3.7) (layer F.SilkS) (width 0.127))
     (pad 1 thru_hole circle (at -5 0 90) (size 2 2) (drill 1.3) (layers *.Cu *.Mask)
-      (net 1 +12V))
+      (net 2 GND))
     (pad 2 thru_hole circle (at 0 0 90) (size 2 2) (drill 1.3) (layers *.Cu *.Mask)
-      (net 2 "Net-(P1-Pad2)"))
+      (net 1 "Net-(P1-Pad2)"))
     (pad 3 thru_hole circle (at 5 0 90) (size 2 2) (drill 1.3) (layers *.Cu *.Mask)
-      (net 2 "Net-(P1-Pad2)"))
+      (net 1 "Net-(P1-Pad2)"))
   )
   (module Socket_Strips:Socket_Strip_Straight_1x02 (layer F.Cu)
@@
     (fp_line (start 3.81 -1.27) (end 3.81 1.27) (layer F.SilkS) (width 0.15))
     (pad 1 thru_hole rect (at 0 0 270) (size 2.032 2.032) (drill 1.016) (layers *.Cu *.Mask F.SilkS)
-      (net 3 GND))
+      (net 2 GND))
     (pad 2 thru_hole oval (at 2.54 0 270) (size 2.032 2.032) (drill 1.016) (layers *.Cu *.Mask F.SilkS)
-      (net 4 "Net-(P2-Pad2)"))
+      (net 3 "Net-(P2-Pad2)"))
     (model Socket_Strips.3dshapes/Socket_Strip_Straight_1x02.wrl
       (at (xyz 0.05 0 0))
@@
       (effects (font (size 1 1) (thickness 0.15)))
     )
-    (fp_text value IPD30N06S2L23ATMA3 (at 0 -2.413) (layer F.Fab) hide
+    (fp_text value IPD30N06S2L-23 (at 0 -2.413) (layer F.Fab) hide
       (effects (font (size 1 1) (thickness 0.15)))
     )
@@
     (fp_line (start 3.429 -9.398) (end 3.429 -7.62) (layer F.SilkS) (width 0.15))
     (pad 1 smd rect (at -2.286 0) (size 1.651 3.048) (layers F.Cu F.Paste F.Mask)
-      (net 5 "Net-(Q1-Pad1)"))
+      (net 4 "Net-(Q1-Pad1)"))
     (pad 2 smd rect (at 0 -6.35) (size 6.096 6.096) (layers F.Cu F.Paste F.Mask)
-      (net 2 "Net-(P1-Pad2)"))
+      (net 1 "Net-(P1-Pad2)"))
     (pad 3 smd rect (at 2.286 0) (size 1.651 3.048) (layers F.Cu F.Paste F.Mask)
-      (net 3 GND))
+      (net 2 GND))
     (model TO_SOT_Packages_SMD.3dshapes/TO-252-2Lead.wrl
       (at (xyz 0 0 0))
@@
     (fp_line (start -0.5 -0.675) (end 0.5 -0.675) (layer F.SilkS) (width 0.15))
     (pad 1 smd rect (at -0.75 0 180) (size 0.5 0.9) (layers F.Cu F.Paste F.Mask)
-      (net 3 GND))
+      (net 2 GND))
     (pad 2 smd rect (at 0.75 0 180) (size 0.5 0.9) (layers F.Cu F.Paste F.Mask)
-      (net 5 "Net-(Q1-Pad1)"))
+      (net 4 "Net-(Q1-Pad1)"))
     (model Resistors_SMD.3dshapes/R_0603.wrl
       (at (xyz 0 0 0))
@@
     (fp_line (start -0.5 -0.675) (end 0.5 -0.675) (layer F.SilkS) (width 0.15))
     (pad 1 smd rect (at -0.75 0 180) (size 0.5 0.9) (layers F.Cu F.Paste F.Mask)
-      (net 5 "Net-(Q1-Pad1)"))
+      (net 4 "Net-(Q1-Pad1)"))
     (pad 2 smd rect (at 0.75 0 180) (size 0.5 0.9) (layers F.Cu F.Paste F.Mask)
-      (net 4 "Net-(P2-Pad2)"))
+      (net 3 "Net-(P2-Pad2)"))
     (model Resistors_SMD.3dshapes/R_0603.wrl
       (at (xyz 0 0 0))
@@
       (rotate (xyz 0 0 0))
     )
+  )
+  (gr_text SIG (at 135.5 104.27) (layer F.SilkS)
+    (effects (font (size 1.5 1.5) (thickness 0.3)))
+  )
+  (gr_text LIGHTS (at 152.5 97.5 90) (layer B.SilkS)
+    (effects (font (size 1.5 1.5) (thickness 0.3)) (justify mirror))
+  )
+  (gr_text GND (at 152.5 105 90) (layer B.SilkS)
+    (effects (font (size 1.5 1.5) (thickness 0.3)) (justify mirror))
+  )
+  (gr_text GND (at 135.5 95.73) (layer F.SilkS)
+    (effects (font (size 1.5 1.5) (thickness 0.3)))
   )
   (gr_text "Designed by Ops" (at 145 100 90) (layer B.SilkS)
@@
   (gr_line (start 155 93) (end 155 107) (layer Edge.Cuts) (width 0.15))
   (gr_line (start 135 91) (end 153 91) (layer Edge.Cuts) (width 0.15))
-  (segment (start 150 95) (end 142.18 95) (width 2) (layer F.Cu) (net 2))
-  (segment (start 142.18 95) (end 141.5 95.68) (width 2) (layer F.Cu) (net 2))
-  (segment (start 150 95) (end 150 100) (width 2) (layer B.Cu) (net 2))
-  (segment (start 150 95) (end 150 100) (width 2) (layer F.Cu) (net 2))
-  (segment (start 138.57 105.1) (end 135 101.53) (width 0.5) (layer F.Cu) (net 4))
-  (segment (start 135 101.53) (end 135 101.27) (width 0.5) (layer F.Cu) (net 4))
-  (segment (start 140.07 105.1) (end 140.07 102.886) (width 0.5) (layer F.Cu) (net 5))
-  (segment (start 140.07 102.886) (end 139.214 102.03) (width 0.5) (layer F.Cu) (net 5))
-  (segment (start 140.07 105.1) (end 142.95 105.1) (width 0.5) (layer F.Cu) (net 5))
-  (zone (net 3) (net_name GND) (layer F.Cu) (hatch edge 0.508)
+  (segment (start 150 95) (end 142.18 95) (width 2) (layer F.Cu) (net 1))
+  (segment (start 142.18 95) (end 141.5 95.68) (width 2) (layer F.Cu) (net 1))
+  (segment (start 150 95) (end 150 100) (width 2) (layer B.Cu) (net 1))
+  (segment (start 150 95) (end 150 100) (width 2) (layer F.Cu) (net 1))
+  (segment (start 138.57 105.1) (end 135 101.53) (width 0.5) (layer F.Cu) (net 3))
+  (segment (start 135 101.53) (end 135 101.27) (width 0.5) (layer F.Cu) (net 3))
+  (segment (start 140.07 105.1) (end 140.07 102.886) (width 0.5) (layer F.Cu) (net 4))
+  (segment (start 140.07 102.886) (end 139.214 102.03) (width 0.5) (layer F.Cu) (net 4))
+  (segment (start 140.07 105.1) (end 142.95 105.1) (width 0.5) (layer F.Cu) (net 4))
+  (zone (net 2) (net_name GND) (layer F.Cu) (hatch edge 0.508)
     (connect_pads (clearance 0.508))
     (min_thickness 0.254)
@@
     )
   )
-  (zone (net 3) (net_name GND) (layer B.Cu) (hatch edge 0.508)
+  (zone (net 2) (net_name GND) (layer B.Cu) (hatch edge 0.508)
     (connect_pads (clearance 0.508))
     (min_thickness 0.254)
