File: Electrical/GotT_Translation_Circuit.sch (KiCad schematic (older format))
At the start: 17 parts, among them P1 Stereo_Audio_Jack_3.5mm, P2 USB_OTG, U1 WT32i, U2 W25Q128FV, U3 MKL04Z32VLC4, U4 MK20DX256VLH7, X1 16 MHz

Commit message: schematic update
Parts:
- removed U3: MKL04Z32VLC4, GotT_Translation_Circuit:NXP_32-LQFP, symbol MKL04Z32VLC4
- added C2, C3: 2.2uF, symbol C_Small
- added C4, C6, C8: 10uF, symbol CP1_Small
- added C5: 0.1uF, symbol C_Small
- added C7: 0.1uF, symbol CP1_Small
- added C9: 01.uF, symbol C_Small
- added D3: D_Small, symbol D_Small
- added D4: Led_Small, symbol Led_Small
- added L1: Ferrite 600, symbol INDUCTOR_SMALL
- added P3: CONN_01X02, symbol CONN_01X02
- added P4: CONN_01X03, symbol CONN_01X03
- added R3, R4: R_Small, symbol R_Small
- added R5: 10K, symbol R_Small
- added SW1: SPST, symbol SPST
- added U3: AP7313, symbol AP7313
- added U5: SGTL5000, symbol SGTL5000
- added U6: MKL04Z32VLC4, symbol MKL04Z32VLC4
- C1: value C_Small -> 0.15uF
Connections:
- net labels added: +12V, +1V8, BCLK, LRCLK, MCLK, MEMCS, MISO, MOSI, RX, SCL, SCLK, SDA, SDCS, TX
- wire segments 26 -> 93
Other:
- note added: "I2S Master"
- note added: "I2S Slave"
- note added: "Power"

Commit message: Schematic update
Parts:
- removed U1: WT32i, GotT_Translation_Circuit:WT32i, symbol WT32i
- added P?: microSD, symbol microSD
- added R?: 10K, symbol R_Small
- added U?: WT32i, symbol WT32i
Connections:
- wire segments 93 -> 99
- no-connect marks 0 -> 2
Other:
- note added: "Audio Codec"
- note added: "Headers"
- note added: "SPI Master"
- note added: "SPI Slave"

Commit message: Schematic update
Parts:
- removed C7: 0.1uF, symbol CP1_Small
- removed D3: D_Small, symbol D_Small
- added C?: 10uF, symbol CP1_Small
- added D?: 1N4749A, symbol ZENERsmall
- added D?: MBRS130L, symbol D_Schottky_Small
- added L?: L_Small, symbol L_Small
- added Q?: FQP47P06, symbol Q_PMOS_GDS
- added R?: 100K, symbol R_Small
- added U?: LM2594, symbol LM2594
- C9: value 01.uF -> 0.1uF
- F1: value FUSE -> 0ZCJ0050AF2E
- P3: value CONN_01X02 -> PWR_IN
- P4: value CONN_01X03 -> PWM_IN
Connections:
- net labels added: VIN
- wire segments 99 -> 117

Commit message: Test board updates
Parts:
- D4: value Led_Small -> PWR LED
- R5: value 10K -> 100
Changed lines of the file:
@@
 U 1 1 57476553
 P 8050 900
-F 0 "F1" H 8150 950 50  0000 C CNN
-F 1 "0ZCJ0050AF2E" H 8050 800 50  0000 C CNN
+F 0 "F1" H 8000 850 50  0000 C CNN
+F 1 "0ZCJ0050AF2E" H 8050 1000 50  0000 C CNN
 F 2 "" H 8050 900 50  0001 C CNN
 F 3 "" H 8050 900 50  0000 C CNN
 	1    8050 900
-	-1   0    0    1
+	1    0    0    -1
 $EndComp
 $Comp
@@
 L Led_Small D4
 U 1 1 5748BC0D
-P 10250 1350
-F 0 "D4" H 10200 1475 50  0000 L CNN
-F 1 "Led_Small" H 10075 1250 50  0000 L CNN
-F 2 "" V 10250 1350 50  0000 C CNN
-F 3 "" V 10250 1350 50  0000 C CNN
-	1    10250 1350
+P 10250 1100
+F 0 "D4" H 10200 1225 50  0000 L CNN
+F 1 "PWR LED" H 10075 1000 50  0000 L CNN
+F 2 "" V 10250 1100 50  0000 C CNN
+F 3 "" V 10250 1100 50  0000 C CNN
+	1    10250 1100
 	0    -1   -1   0
 $EndComp
@@
 L R_Small R5
 U 1 1 5748BD56
-P 10250 1100
-F 0 "R5" H 10280 1120 50  0000 L CNN
-F 1 "10K" H 10280 1060 50  0000 L CNN
-F 2 "" H 10250 1100 50  0001 C CNN
-F 3 "" H 10250 1100 50  0000 C CNN
-	1    10250 1100
-	1    0    0    -1
-$EndComp
+P 10250 1350
+F 0 "R5" H 10280 1370 50  0000 L CNN
+F 1 "100" H 10280 1310 50  0000 L CNN
+F 2 "" H 10250 1350 50  0001 C CNN
+F 3 "" H 10250 1350 50  0000 C CNN
+	1    10250 1350
+	1    0    0    -1
+$EndComp

Commit message: Schematic, documentation update
Parts:
- removed U4: MK20DX256VLH7, GotT_Translation_Circuit:NXP_64-LQFP, symbol MK20DX256VLH7
- removed U6: MKL04Z32VLC4, symbol MKL04Z32VLC4
- removed X1: 16 MHz, symbol NX2520SA
- added P1: LIGHTS_HEADER, symbol CONN_01X03
- added Q2: IPD30N06S2L-23, symbol Q_NMOS_GDS
- added R3: 100R, symbol R_Small
- added R4: 10K, symbol R_Small
- added R5: 220R, symbol R_Small
- added R6: ???, symbol R_Small
- added U2: SN74LVC1G34, symbol SN74LVC1G34
- added U3: FOD817D3SD, symbol FOD817D3SD
- R2: renamed from R5; value 100 -> 100R
- gave numbers to parts that had none: 7
- renumbered C8 to C2, C9 to C3, D4 to D3, P4 to P2
Connections:
- net labels added: GNDD, ISOLATED_PWM, LIGHTS
- net labels removed: RESET
- wire segments 117 -> 112
Other:
- note removed: "I2S Master"
- note removed: "SPI Master"

Commit message: Combine sub-circuits, update BOM/lib, add PDFs
Parts:
- removed P2: USB_OTG, symbol USB_OTG
- removed U?: WT32i, symbol WT32i
- added C?: 2.2uF, symbol C_Small
- added P?: CONN_01X06, symbol CONN_01X06
- added U7: Teensy3.2, symbol Teensy3.2
- added U8: WT32i, symbol WT32i
- D4: renamed from D2; value Led_Small -> CONN_LED
- L1: renamed from L2; value L_Small -> 115uH
- R2: value 100R -> 820R
- R9: renamed from R2; value R_Small -> 100R
- gave numbers to parts that had none: 2
- renumbered C2 to C4, C3 to C5, C5 to C6, C1 to C7, L1 to L2, P3 to P1, P1 to P2, P2 to P3, R1 to R8, U3 to U4, U2 to U6
Connections:
- net labels added: UART_RXD, UART_TXD, VOL
- wire segments 112 -> 150
- no-connect marks 2 -> 5
Other:
- note added: "AUDIO CODEC"
- note added: "BLUETOOTH"
- note added: "LIGHTS"
- note added: "MEMORY"
- note added: "POWER"
- note added: "PWM ISOLATOR"
- note added: "TEENSY"
- note removed: "Audio Codec"
- note removed: "Headers"
- note removed: "Memory"
- note removed: "Power"
- note removed: "Wireless"

Commit message: schematic updates
Parts:
- removed D1: 1N4749A, symbol ZENERsmall
- removed F1: 0ZCJ0050AF2E, symbol FUSE
- removed L2: Ferrite 600, symbol INDUCTOR_SMALL
- removed SW1: SPST, symbol SPST
- added D1: 1N4749A, symbol D_Zener_Small_ALT
- added F1: 0ZCJ0050AF2E, symbol Polyfuse
- added L2: Ferrite 600, symbol Ferrite_Bead_Small
- added R? (x2): 2.2K, symbol R_Small
- added SW1: PWR_SPST, symbol SW_SPST
- D3, D4: symbol Led_Small -> LED_Small
- P1: symbol CONN_01X02 -> Conn_01x02
- P2, P3: symbol CONN_01X03 -> Conn_01x03
- P?: value CONN_01X06 -> UART_CONN; symbol CONN_01X06 -> Conn_01x06
Connections:
- net labels added: TRIM1, TRIM2, TRIM3
- wire segments 150 -> 174
- no-connect marks 5 -> 16
Other:
- note added: "PWM ISOLATE"
- note removed: "PWM ISOLATOR"
